File: pcb/headstage-16stim.kicad_sch (KiCad schematic)
At the start: 8 parts, among them J1 OE_COAX-ADAPTER-XFL-A (DNP), J2 DF40C-70DP-0.4V(51)

Commit message: Revision B
- Bring in changes from headstage-rhs116 rev. C that should make this design
  fully functional
Parts:
- added TP5: GPIO2, jonnew:TestPoint_Pad_D0.6mm, symbol Connector:TestPoint
Connections:
- new net FPGA/GPIO2_{Ser}: TP5.1
- no-connect marks 52 -> 53
Other:
- sheet FPGA ports: added GPIO2_{Ser}; removed none
- sheet Serializer ports: added GPIO1, GPIO2; removed none
- moved on the sheet: TP2
