File: pcb/power.kicad_sch (KiCad schematic)
At the start: 35 parts, among them U10 NCP163AFCT120T2G, U13 TPS826951, U4 LTC3265xxHC#PBF, U5 NCP163AFCT180T2G, U9 NCP163AFCT330T2G

Commit message: Revision B
- Bring in changes from headstage-rhs116 rev. C that should make this design
  fully functional
Parts:
- added R5, R6: 124k,1%, Resistor_SMD:R_0201_0603Metric, symbol Device:R_US
- R19, R23: value 125k,1% -> 124k,1%
Connections:
- net +4V: no longer U9.B1 (EN)
- net +7V: now also R5.2
- net GND: now also R6.1
- new net 3v3_{EN}: R5.1, R6.2, U9.B1 (EN)
